Commit message: added gazebo plugin

File: urdf/robot_structure.xacro (robot description, xacro)
@@ -1,4 +1,5 @@
 <?xml version="1.0" ?>
 <robot xmlns:xacro="http://www.ros.org/wiki/xacro">
+    <link name="base_footprint" />
     <link name="base_link">
         <inertial>
@@ -81,4 +82,9 @@
         </collision>
     </link>
+    <joint name="base_footprint" type="fixed">
+        <parent link="base_footprint" />
+        <child link="base_link" />
+        <origin xyz="0 0 0" rpy="0 0 0" />
+    </joint>
     <joint name="base_right_wheel_joint" type="continuous">
         <origin xyz="0.0 -0.1 0.05" rpy="0 0 0"/>
